Commit message: Working rover sim: SLAM + Nav2 on flat ground, dual-lidar traversability experiment (unfinished,not working)

File: src/forros_description/urdf/forros.xacro (robot description, xacro)
@@ -7,6 +7,6 @@
   <inertial>
     <origin xyz="0.1099999999999859 0.115 0.12499999999999567" rpy="0 0 0"/>
-    <mass value="42.38938346244173"/>
-    <inertia ixx="0.169907" iyy="0.346538" izz="0.459219" ixy="-0.0" iyz="-0.0" ixz="0.0"/>
+    <mass value="4.238938346244173"/>
+    <inertia ixx="0.0169907" iyy="0.0346538" izz="0.0459219" ixy="-0.0" iyz="-0.0" ixz="0.0"/>
   </inertial>
   <visual>
@@ -27,6 +27,6 @@
   <inertial>
     <origin xyz="1.0320994585366616e-07 0.02500000022351742 4.163336342344337e-17" rpy="0 0 0"/>
-    <mass value="3.313045200437847"/>
-    <inertia ixx="0.002916" iyy="0.004451" izz="0.002916" ixy="0.0" iyz="0.0" ixz="-0.0"/>
+    <mass value="0.3313045200437847"/>
+    <inertia ixx="0.0002916" iyy="0.0004451" izz="0.0002916" ixy="0.0" iyz="0.0" ixz="-0.0"/>
   </inertial>
   <visual>
@@ -47,6 +47,6 @@
   <inertial>
     <origin xyz="1.0320994585366616e-07 -0.025000000223517366 9.71445146547012e-17" rpy="0 0 0"/>
-    <mass value="3.313045200437847"/>
-    <inertia ixx="0.002916" iyy="0.004451" izz="0.002916" ixy="0.0" iyz="0.0" ixz="0.0"/>
+    <mass value="0.3313045200437847"/>
+    <inertia ixx="0.0002916" iyy="0.0004451" izz="0.0002916" ixy="0.0" iyz="0.0" ixz="0.0"/>
   </inertial>
   <visual>
@@ -127,6 +127,6 @@
   <inertial>
     <origin xyz="3.2278066333657485e-07 0.025000000067055467 4.163336342344337e-17" rpy="0 0 0"/>
-    <mass value="3.313045200437847"/>
-    <inertia ixx="0.002916" iyy="0.004451" izz="0.002916" ixy="-0.0" iyz="0.0" ixz="-0.0"/>
+    <mass value="0.3313045200437847"/>
+    <inertia ixx="0.0002916" iyy="0.0004451" izz="0.0002916" ixy="-0.0" iyz="0.0" ixz="-0.0"/>
   </inertial>
   <visual>
@@ -147,6 +147,6 @@
   <inertial>
     <origin xyz="1.032099458120328e-07 0.025000000223517643 4.163336342344337e-17" rpy="0 0 0"/>
-    <mass value="3.313045200437847"/>
-    <inertia ixx="0.002916" iyy="0.004451" izz="0.002916" ixy="-0.0" iyz="0.0" ixz="-0.0"/>
+    <mass value="0.3313045200437847"/>
+    <inertia ixx="0.0002916" iyy="0.0004451" izz="0.0002916" ixy="-0.0" iyz="0.0" ixz="-0.0"/>
   </inertial>
   <visual>
@@ -167,6 +167,6 @@
   <inertial>
     <origin xyz="3.2278066333657485e-07 -0.02500000006705523 4.85722573273506e-17" rpy="0 0 0"/>
-    <mass value="3.313045200437847"/>
-    <inertia ixx="0.002916" iyy="0.004451" izz="0.002916" ixy="0.0" iyz="0.0" ixz="0.0"/>
+    <mass value="0.3313045200437847"/>
+    <inertia ixx="0.0002916" iyy="0.0004451" izz="0.0002916" ixy="0.0" iyz="0.0" ixz="0.0"/>
   </inertial>
   <visual>
@@ -187,6 +187,6 @@
   <inertial>
     <origin xyz="1.0320994583978838e-07 -0.025000000223517435 4.163336342344337e-17" rpy="0 0 0"/>
-    <mass value="3.313045200437847"/>
-    <inertia ixx="0.002916" iyy="0.004451" izz="0.002916" ixy="0.0" iyz="0.0" ixz="0.0"/>
+    <mass value="0.3313045200437847"/>
+    <inertia ixx="0.0002916" iyy="0.0004451" izz="0.0002916" ixy="0.0" iyz="0.0" ixz="0.0"/>
   </inertial>
   <visual>
@@ -348,5 +348,6 @@
   <parent link="motor_house_right_mid_1"/>
   <child link="right_mid_wheel_1"/>
-  <axis xyz="-0.0 1.0 0.0"/>
+  <axis xyz="-0.0 -1.0 0.0"/>
+  <limit effort="10.0" velocity="20.0"/>
 </joint>
 <joint name="left_mid_wheel" type="continuous">
@@ -354,5 +355,6 @@
   <parent link="motor_house_left_mid_1"/>
   <child link="left_mid_wheel_1"/>
-  <axis xyz="-0.0 1.0 0.0"/>
+  <axis xyz="-0.0 -1.0 0.0"/>
+  <limit effort="10.0" velocity="20.0"/>
 </joint>
 <joint name="left_rocker_bogie" type="revolute">
@@ -362,4 +364,5 @@
   <axis xyz="-0.0 1.0 0.0"/>
   <limit upper="0.872665" lower="-0.436332" effort="100" velocity="100"/>
+  <dynamics damping="0.1" friction="0.5"/>
 </joint>
 <joint name="Rigid 58" type="fixed">
@@ -374,4 +377,5 @@
   <axis xyz="-0.0 1.0 0.0"/>
   <limit upper="0.872665" lower="-0.436332" effort="100" velocity="100"/>
+  <dynamics damping="0.1" friction="0.5"/>
 </joint>
 <joint name="right_back_wheel" type="continuous">
@@ -379,5 +383,6 @@
   <parent link="motor_house_right_back_2"/>
   <child link="right_back_wheel_1"/>
-  <axis xyz="0.0 1.0 0.0"/>
+  <axis xyz="0.0 -1.0 0.0"/>
+  <limit effort="10.0" velocity="20.0"/>
 </joint>
 <joint name="right_front_wheel" type="continuous">
@@ -385,5 +390,6 @@
   <parent link="motor_house_right_front_1"/>
   <child link="right_front_wheel_1"/>
-  <axis xyz="0.0 1.0 0.0"/>
+  <axis xyz="0.0 -1.0 0.0"/>
+  <limit effort="10.0" velocity="20.0"/>
 </joint>
 <joint name="left_back_wheel" type="continuous">
@@ -391,5 +397,6 @@
   <parent link="motor_house_left_back_1"/>
   <child link="left_back_wheel_1"/>
-  <axis xyz="-0.0 1.0 -0.0"/>
+  <axis xyz="-0.0 -1.0 -0.0"/>
+  <limit effort="10.0" velocity="20.0"/>
 </joint>
 <joint name="left_front_wheel" type="continuous">
@@ -397,5 +404,6 @@
   <parent link="motor_house_left_front_1"/>
   <child link="left_front_wheel_1"/>
-  <axis xyz="-0.0 1.0 -0.0"/>
+  <axis xyz="-0.0 -1.0 -0.0"/>
+  <limit effort="10.0" velocity="20.0"/>
 </joint>
 <joint name="Rigid 67" type="fixed">
@@ -438,4 +446,5 @@
   <axis xyz="0.0 -1.0 0.0"/>
   <limit upper="0.349066" lower="-0.349066" effort="100" velocity="100"/>
+  <dynamics damping="0.1" friction="0.5"/>
 </joint>
 <joint name="right_rocker_arm" type="revolute">
@@ -445,4 +454,50 @@
   <axis xyz="0.0 1.0 0.0"/>
   <limit upper="0.349066" lower="-0.349066" effort="100" velocity="100"/>
+  <dynamics damping="0.1" friction="0.5"/>
+  <mimic joint="left_rocker_arm" multiplier="1" offset="0"/>
+</joint>
+<link name="lidar_link">
+  <inertial>
+    <mass value="0.11"/>
+    <inertia ixx="1e-5" iyy="1e-5" izz="1e-5" ixy="0" iyz="0" ixz="0"/>
+  </inertial>
+  <visual>
+    <geometry>
+      <cylinder radius="0.0278" length="0.0413"/>
+    </geometry>
+    <material name="silver"/>
+  </visual>
+  <collision>
+    <geometry>
+      <cylinder radius="0.0278" length="0.0413"/>
+    </geometry>
+  </collision>
+</link>
+<joint name="lidar_joint" type="fixed">
+  <origin xyz="-0.0102 0.115 0.18" rpy="0 0 0"/>
+  <parent link="base_link"/>
+  <child link="lidar_link"/>
+</joint>
+<link name="lidar_link_tilt">
+  <inertial>
+    <mass value="0.11"/>
+    <inertia ixx="1e-5" iyy="1e-5" izz="1e-5" ixy="0" iyz="0" ixz="0"/>
+  </inertial>
+  <visual>
+    <geometry>
+      <cylinder radius="0.0278" length="0.0413"/>
+    </geometry>
+    <material name="silver"/>
+  </visual>
+  <collision>
+    <geometry>
+      <cylinder radius="0.0278" length="0.0413"/>
+    </geometry>
+  </collision>
+</link>
+<joint name="lidar_joint_tilt" type="fixed">
+  <origin xyz="-0.08 0.115 0.12" rpy="0 -0.6109 0"/>
+  <parent link="base_link"/>
+  <child link="lidar_link_tilt"/>
 </joint>
 </robot>

Commit message: Revert to single horizontal lidar - remove tilted lidar/traversability experiment

File: src/forros_description/urdf/forros.xacro (robot description, xacro)
@@ -479,25 +479,3 @@
   <child link="lidar_link"/>
 </joint>
-<link name="lidar_link_tilt">
-  <inertial>
-    <mass value="0.11"/>
-    <inertia ixx="1e-5" iyy="1e-5" izz="1e-5" ixy="0" iyz="0" ixz="0"/>
-  </inertial>
-  <visual>
-    <geometry>
-      <cylinder radius="0.0278" length="0.0413"/>
-    </geometry>
-    <material name="silver"/>
-  </visual>
-  <collision>
-    <geometry>
-      <cylinder radius="0.0278" length="0.0413"/>
-    </geometry>
-  </collision>
-</link>
-<joint name="lidar_joint_tilt" type="fixed">
-  <origin xyz="-0.08 0.115 0.12" rpy="0 -0.6109 0"/>
-  <parent link="base_link"/>
-  <child link="lidar_link_tilt"/>
-</joint>
 </robot>

Commit message: Added depth camera

File: src/forros_description/urdf/forros.xacro (robot description, xacro)
@@ -446,5 +446,5 @@
   <axis xyz="0.0 -1.0 0.0"/>
   <limit upper="0.349066" lower="-0.349066" effort="100" velocity="100"/>
-  <dynamics damping="0.1" friction="0.5"/>
+  <dynamics damping="2" friction="0.5"/>
 </joint>
 <joint name="right_rocker_arm" type="revolute">
@@ -454,5 +454,5 @@
   <axis xyz="0.0 1.0 0.0"/>
   <limit upper="0.349066" lower="-0.349066" effort="100" velocity="100"/>
-  <dynamics damping="0.1" friction="0.5"/>
+  <dynamics damping="2" friction="0.5"/>
   <mimic joint="left_rocker_arm" multiplier="1" offset="0"/>
 </joint>
@@ -479,3 +479,25 @@
   <child link="lidar_link"/>
 </joint>
+<link name="camera_link">
+  <inertial>
+    <mass value="0.072"/>
+    <inertia ixx="1e-5" iyy="1e-5" izz="1e-5" ixy="0" iyz="0" ixz="0"/>
+  </inertial>
+  <visual>
+    <geometry>
+      <box size="0.025 0.09 0.025"/>
+    </geometry>
+    <material name="silver"/>
+  </visual>
+  <collision>
+    <geometry>
+      <box size="0.025 0.09 0.025"/>
+    </geometry>
+  </collision>
+</link>
+<joint name="camera_joint" type="fixed">
+  <origin xyz="-0.04 0.115 0.12" rpy="3.14159 -3.14159 0"/>
+  <parent link="base_link"/>
+  <child link="camera_link"/>
+</joint>
 </robot>
